File: nixiesp.kicad_pcb (KiCad board)
At the start: 2 copper layers, 152.4 x 53.3 mm, 50 parts, among them J1 Power 9-15V, J2 ESP8266, J3 Nixie PSU low, J4 CONN_01X02, Q1 BS107, Q2 BS107, Q3 BS107, Q4 BS107, U1 74HC595, U10 LM1117-3.3, U2 K155ID1, U3 K155ID1, U4 K155ID1, U5 74HC595, U6 K155ID1, U7 K155ID1, U8 74HC595, U9 74141-DIP

Commit message: Rotate tubes and other fixes
Parts:
- added U11: LM1117-3.3, TO_SOT_Packages_SMD:SOT-223, B.Cu at (129.5, 97.8)
- U10: moved to B.Cu
- U9: value 74141-DIP -> K155ID1
- moved J4 45.7 mm to (228.6, 111.8)
- moved U10 26.2 mm to (180.3, 97.8)
- moved R11 18.0 mm to (228.6, 73.7), turned to 180 degrees
- moved R12 18.0 mm to (205.7, 73.7), turned to 180 degrees
- moved R13 18.0 mm to (177.8, 73.7), turned to 180 degrees
- moved R14 18.0 mm to (154.9, 73.7), turned to 180 degrees
- moved R15 18.0 mm to (127.0, 73.7), turned to 180 degrees
- moved R16 18.0 mm to (104.1, 73.7), turned to 180 degrees
- moved R2 12.5 mm to (146.1, 73.7), turned to 180 degrees
- moved R3 12.5 mm to (95.2, 73.7), turned to 180 degrees
- moved R4 12.5 mm to (168.9, 73.7), turned to 180 degrees
- moved R5 12.5 mm to (196.8, 73.7), turned to 180 degrees
- moved R6 12.5 mm to (219.7, 73.7), turned to 180 degrees
- moved R1 12.5 mm to (118.1, 73.7), turned to 180 degrees
- moved N10 10.2 mm to (129.5, 90.2), turned to 270 degrees
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Connections:
- J2 pad 6: (no net) -> VCC
- U2 pad 1: Net-(N5-Pad0) -> Net-(N5-Pad4)
- U2 pad 10: Net-(N5-Pad3) -> Net-(N5-Pad9)
- U2 pad 11: Net-(N5-Pad4) -> Net-(N5-Pad7)
- U2 pad 13: Net-(N5-Pad5) -> Net-(N5-Pad6)
- U2 pad 14: Net-(N5-Pad6) -> Net-(N5-Pad1)
- U2 pad 15: Net-(N5-Pad7) -> Net-(N5-Pad3)
- U2 pad 16: Net-(N5-Pad8) -> Net-(N5-Pad5)
- U2 pad 2: Net-(N5-Pad9) -> Net-(N5-Pad2)
- U2 pad 8: Net-(N5-Pad1) -> Net-(N5-Pad8)
- U2 pad 9: Net-(N5-Pad2) -> Net-(N5-Pad0)
- U3 pad 1: Net-(N6-Pad0) -> Net-(N6-Pad4)
- U3 pad 10: Net-(N6-Pad3) -> (no net)
- U3 pad 11: Net-(N6-Pad4) -> Net-(N6-Pad7)
- U3 pad 13: Net-(N6-Pad5) -> Net-(N6-Pad6)
- U3 pad 14: Net-(N6-Pad6) -> Net-(N6-Pad1)
- U3 pad 15: Net-(N6-Pad7) -> Net-(N6-Pad3)
- U3 pad 16: (no net) -> Net-(N6-Pad5)
- U3 pad 2: (no net) -> Net-(N6-Pad2)
- U3 pad 8: Net-(N6-Pad1) -> (no net)
- U3 pad 9: Net-(N6-Pad2) -> Net-(N6-Pad0)
- U4 pad 1: Net-(N3-Pad0) -> Net-(N3-Pad4)
- U4 pad 10: Net-(N3-Pad3) -> Net-(N3-Pad9)
- U4 pad 11: Net-(N3-Pad4) -> Net-(N3-Pad7)
- U4 pad 13: Net-(N3-Pad5) -> Net-(N3-Pad6)
- U4 pad 14: Net-(N3-Pad6) -> Net-(N3-Pad1)
- U4 pad 15: Net-(N3-Pad7) -> Net-(N3-Pad3)
- U4 pad 16: Net-(N3-Pad8) -> Net-(N3-Pad5)
- U4 pad 2: Net-(N3-Pad9) -> Net-(N3-Pad2)
- U4 pad 8: Net-(N3-Pad1) -> Net-(N3-Pad8)
- U4 pad 9: Net-(N3-Pad2) -> Net-(N3-Pad0)
- U6 pad 1: Net-(N4-Pad0) -> Net-(N4-Pad4)
- U6 pad 10: Net-(N4-Pad3) -> (no net)
- U6 pad 11: Net-(N4-Pad4) -> Net-(N4-Pad7)
- U6 pad 13: Net-(N4-Pad5) -> Net-(N4-Pad6)
- U6 pad 14: Net-(N4-Pad6) -> Net-(N4-Pad1)
- U6 pad 15: Net-(N4-Pad7) -> Net-(N4-Pad3)
- U6 pad 16: (no net) -> Net-(N4-Pad5)
- U6 pad 2: (no net) -> Net-(N4-Pad2)
- U6 pad 8: Net-(N4-Pad1) -> (no net)
- U6 pad 9: Net-(N4-Pad2) -> Net-(N4-Pad0)
- U7 pad 1: Net-(N1-Pad0) -> Net-(N1-Pad4)
- U7 pad 10: Net-(N1-Pad3) -> Net-(N1-Pad9)
- U7 pad 11: Net-(N1-Pad4) -> Net-(N1-Pad7)
- U7 pad 13: Net-(N1-Pad5) -> Net-(N1-Pad6)
- U7 pad 14: Net-(N1-Pad6) -> Net-(N1-Pad1)
- U7 pad 15: Net-(N1-Pad7) -> Net-(N1-Pad3)
- U7 pad 16: Net-(N1-Pad8) -> Net-(N1-Pad5)
- U7 pad 2: Net-(N1-Pad9) -> Net-(N1-Pad2)
- U7 pad 8: Net-(N1-Pad1) -> Net-(N1-Pad8)
- U7 pad 9: Net-(N1-Pad2) -> Net-(N1-Pad0)
- U9 pad 1: Net-(N2-Pad0) -> (no net)
- U9 pad 10: Net-(N2-Pad3) -> (no net)
- U9 pad 14: (no net) -> Net-(N2-Pad1)
- U9 pad 15: (no net) -> Net-(N2-Pad3)
- U9 pad 2: (no net) -> Net-(N2-Pad2)
- U9 pad 8: Net-(N2-Pad1) -> (no net)
- U9 pad 9: Net-(N2-Pad2) -> Net-(N2-Pad0)
Routing:
- net Net-(J1-Pad1): track 192.8 -> 246.7 mm
- net Net-(N1-Pad1): track 31.8 -> 4.78 mm
- net Net-(N3-Pad1): track 31.8 -> 4.78 mm
- net Net-(N6-Pad1): track 31.8 -> 4.78 mm
- net Net-(N4-Pad1): track 31.8 -> 4.78 mm
- net Net-(N2-Pad1): track 30.9 -> 4.78 mm
- net Net-(N5-Pad1): track 30.8 -> 4.78 mm
- net VCC: track 270.4 -> 249.3 mm
- net Net-(J4-Pad1): track 189.9 -> 210.1 mm
- net Net-(N1-Pad0): track 27.2 -> 9.50 mm
- net Net-(N3-Pad0): track 27.2 -> 9.50 mm
- net Net-(N5-Pad0): track 27.2 -> 9.50 mm
- net Net-(N1-PadA): track 2.95 -> 20.4 mm
- net Net-(N2-PadA): track 2.95 -> 20.4 mm
- net Net-(N3-Pad5): track 7.22 -> 24.6 mm
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
Commit message: Hopefully final changes
Parts:
- removed D1, D10, D2, D3, D4, D9: LED, LEDs:LED_D5.0mm
- removed R1, R2, R3, R4, R5, R6: 330, Resistors_THT:R_Axial_DIN0204_L3.6mm_D1.6mm_P5.08mm_Horizontal
- added J10: CONN_01X06, Pin_Headers:Pin_Header_Angled_1x06_Pitch2.54mm, F.Cu at (101.6, 66.0)
- added J11: CONN_01X06, Pin_Headers:Pin_Header_Angled_1x06_Pitch2.54mm, F.Cu at (124.5, 66.0)
- added J12: CONN_01X06, Pin_Headers:Pin_Header_Angled_1x06_Pitch2.54mm, F.Cu at (152.4, 66.0)
- added J13: CONN_01X07, Pin_Headers:Pin_Header_Angled_1x07_Pitch2.54mm, F.Cu at (177.8, 66.0)
- added J14: CONN_01X02, Pin_Headers:Pin_Header_Angled_1x02_Pitch2.54mm, F.Cu at (78.7, 66.0)
- added J15: CONN_01X01, Connectors:1pin, B.Cu at (148.6, 43.2)
- added J16: CONN_01X01, Connectors:1pin, B.Cu at (69.8, 43.2)
- added J17: CONN_01X01, Connectors:1pin, B.Cu at (171.4, 43.2)
- added J18: CONN_01X01, Connectors:1pin, B.Cu at (120.7, 43.2)
- added J19: CONN_01X01, Connectors:1pin, B.Cu at (47.0, 43.2)
- added J20: CONN_01X01, Connectors:1pin, B.Cu at (97.8, 43.2)
- added J21: CONN_01X01, Connectors:1pin, B.Cu at (188.0, 121.9)
- added J22: CONN_01X01, Connectors:1pin, B.Cu at (30.5, 68.6)
- added J23: CONN_01X01, Connectors:1pin, B.Cu at (30.5, 121.9)
- added J24: CONN_01X01, Connectors:1pin, B.Cu at (188.0, 86.4)
- added J25: CONN_01X01, Connectors:1pin, B.Cu at (30.5, 86.4)
- added J26: CONN_01X02, Pin_Headers:Pin_Header_Angled_1x02_Pitch2.54mm, F.Cu at (129.5, 66.0)
- added J27: CONN_01X06, Socket_Strips:Socket_Strip_Straight_1x06_Pitch2.54mm, B.Cu at (50.8, 90.4)
- added J28: CONN_01X06, Socket_Strips:Socket_Strip_Straight_1x06_Pitch2.54mm, B.Cu at (73.7, 90.4)
- added J29: CONN_01X06, Socket_Strips:Socket_Strip_Straight_1x06_Pitch2.54mm, B.Cu at (101.6, 90.4)
- added J30: CONN_01X06, Socket_Strips:Socket_Strip_Straight_1x06_Pitch2.54mm, B.Cu at (124.5, 90.4)
- added J31: CONN_01X07, Socket_Strips:Socket_Strip_Straight_1x07_Pitch2.54mm, B.Cu at (177.8, 90.4)
- added J32: CONN_01X02, Socket_Strips:Socket_Strip_Straight_1x02_Pitch2.54mm, B.Cu at (76.2, 90.4)
- added J33: CONN_01X02, Socket_Strips:Socket_Strip_Straight_1x02_Pitch2.54mm, B.Cu at (127.0, 90.4)
- added J5: CONN_01X06, Socket_Strips:Socket_Strip_Straight_1x06_Pitch2.54mm, B.Cu at (152.4, 90.4)
- added J6: CONN_01X01, Connectors:1pin, B.Cu at (188.0, 68.6)
- added J7: CONN_01X01, Connectors:1pin, B.Cu at (188.0, 33.0)
- added J8: CONN_01X01, Connectors:1pin, B.Cu at (30.5, 33.0)
- added J9: CONN_01X05, Socket_Strips:Socket_Strip_Straight_1x05_Pitch2.54mm, B.Cu at (177.8, 113.3)
- added U12: LM1117-3.3, TO_SOT_Packages_SMD:SOT-223, F.Cu at (134.6, 119.4)
- added U13: 74HC595, Housings_DIP:DIP-16_W7.62mm, B.Cu at (68.6, 104.4)
- added U14: 74HC595, Housings_DIP:DIP-16_W7.62mm, B.Cu at (154.9, 104.4)
- J1: footprint Connectors:BARREL_JACK -> Connectors_Terminal_Blocks:TerminalBlock_Pheonix_PT-3.5mm_2pol; moved to B.Cu
- J2, N1, N10, N2, N3, N4, N5, N6, N7, N8, N9, U1, U2, U3, U4, U5, U6, U7, U8, U9: moved to B.Cu
- J3: value Nixie PSU low -> CONN_01X06; footprint Pin_Headers:Pin_Header_Straight_1x02_Pitch2.54mm -> Pin_Headers:Pin_Header_Angled_1x06_Pitch2.54mm
- J4: value CONN_01X02 -> CONN_01X06; footprint Pin_Headers:Pin_Header_Straight_1x02_Pitch2.54mm -> Pin_Headers:Pin_Header_Angled_1x06_Pitch2.54mm
- Q1, Q2, Q3, Q4: footprint TO_SOT_Packages_THT:TO-92_Molded_Narrow -> TO_SOT_Packages_THT:TO-92_Inline_Wide; moved to B.Cu
- R10, R11, R12, R13, R14, R15, R16, R7, R8, R9: footprint Resistors_THT:R_Axial_DIN0204_L3.6mm_D1.6mm_P5.08mm_Horizontal -> Resistors_THT:R_Axial_DIN0207_L6.3mm_D2.5mm_P7.62mm_Horizontal; moved to B.Cu
- U10: value LM1117-3.3 -> LM1117-5.0; moved to F.Cu
- U11: value LM1117-3.3 -> 74HC595; footprint TO_SOT_Packages_SMD:SOT-223 -> Housings_DIP:DIP-16_W7.62mm
- moved R11 197.1 mm to (36.8, 27.9), turned to 270 degrees
- moved J2 179.8 mm to (41.9, 113.3), turned to 0 degrees
- moved N5 175.3 mm to (47.0, 43.2), turned to 180 degrees
- moved U8 166.4 mm to (47.0, 104.4)
- moved J4 161.5 mm to (73.7, 66.0), turned to 270 degrees
- moved U2 158.1 mm to (55.9, 63.5)
- moved R12 153.0 mm to (59.7, 27.9), turned to 270 degrees
- moved N6 131.3 mm to (69.8, 43.2), turned to 180 degrees
- moved U3 114.6 mm to (78.7, 63.5)
- moved Q1 113.1 mm to (85.1, 66.0), turned to 270 degrees
- moved R7 110.3 mm to (85.1, 55.9), turned to 270 degrees
- moved R8 110.3 mm to (82.5, 55.9), turned to 270 degrees
- moved N9 109.7 mm to (83.8, 38.1), turned to 90 degrees
- moved U9 105.2 mm to (180.3, 63.5)
- moved Q2 103.9 mm to (82.5, 66.0), turned to 270 degrees
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Connections:
- net Net-(J2-Pad3) renamed /data
- J1 pad 1: Net-(J1-Pad1) -> GND
- J1 pad 2: GND -> Net-(J1-Pad2)
- J2 pad 5: Net-(J2-Pad5) -> /latch
- J2 pad 7: Net-(J2-Pad7) -> /clock
- J3 pad 1: Net-(J1-Pad1) -> Net-(J3-Pad1)
- J3 pad 2: GND -> Net-(J3-Pad2)
- J4 pad 2: GND -> Net-(J4-Pad2)
- N10 pad A: Net-(J4-Pad1) -> Net-(J13-Pad1)
- N2 pad 4: (no net) -> Net-(N2-Pad4)
- N2 pad 5: (no net) -> Net-(N2-Pad5)
- N2 pad 6: (no net) -> Net-(N2-Pad6)
- N2 pad 7: (no net) -> Net-(N2-Pad7)
- N2 pad 8: (no net) -> Net-(N2-Pad8)
- N2 pad 9: (no net) -> Net-(N2-Pad9)
- N4 pad 8: (no net) -> Net-(N4-Pad8)
- N4 pad 9: (no net) -> Net-(N4-Pad9)
- N6 pad 8: (no net) -> Net-(N6-Pad8)
- N6 pad 9: (no net) -> Net-(N6-Pad9)
- N7 pad A: Net-(J4-Pad1) -> Net-(J13-Pad1)
- N8 pad A: Net-(J4-Pad1) -> Net-(J13-Pad1)
- N9 pad A: Net-(J4-Pad1) -> Net-(J13-Pad1)
- Q1 pad 2: Net-(Q1-Pad2) -> Net-(J14-Pad2)
- Q2 pad 2: Net-(Q2-Pad2) -> Net-(J14-Pad1)
- Q3 pad 2: Net-(Q3-Pad2) -> Net-(J26-Pad2)
- Q4 pad 2: Net-(Q4-Pad2) -> Net-(J26-Pad1)
- R11 pad 1: Net-(J4-Pad1) -> Net-(J13-Pad1)
- R12 pad 1: Net-(J4-Pad1) -> Net-(J13-Pad1)
- R13 pad 1: Net-(J4-Pad1) -> Net-(J13-Pad1)
- R14 pad 1: Net-(J4-Pad1) -> Net-(J13-Pad1)
- R15 pad 1: Net-(J4-Pad1) -> Net-(J13-Pad1)
- R16 pad 1: Net-(J4-Pad1) -> Net-(J13-Pad1)
- U1 pad 1: Net-(U1-Pad1) -> Net-(J33-Pad1)
- U1 pad 11: Net-(J2-Pad7) -> /clock
- U1 pad 12: Net-(J2-Pad5) -> /latch
- U1 pad 15: Net-(U1-Pad15) -> (no net)
- U1 pad 2: Net-(U1-Pad2) -> Net-(J33-Pad2)
- U1 pad 3: Net-(U1-Pad3) -> Net-(J5-Pad5)
- U1 pad 4: Net-(Q3-Pad2) -> Net-(J5-Pad4)
- U1 pad 5: Net-(U1-Pad5) -> Net-(J5-Pad2)
- U1 pad 6: Net-(Q4-Pad2) -> Net-(J5-Pad1)
- U1 pad 7: Net-(U1-Pad7) -> (no net)
- U1 pad 9: (no net) -> Net-(U1-Pad9)
- U10 pad 3: Net-(J1-Pad1) -> Net-(J1-Pad2)
- U11 pad 1: GND -> (no net)
- U11 pad 2: VCC -> (no net)
- U11 pad 3: Net-(J1-Pad1) -> Net-(J30-Pad5)
- U11 pad 4: VCC -> Net-(J30-Pad4)
- U2 pad 1: Net-(N5-Pad4) -> Net-(N5-Pad5)
- U2 pad 10: Net-(N5-Pad9) -> Net-(N5-Pad0)
- U2 pad 16: Net-(N5-Pad5) -> Net-(N5-Pad4)
- U2 pad 3: Net-(U2-Pad3) -> Net-(J3-Pad1)
- U2 pad 4: Net-(U2-Pad4) -> Net-(J3-Pad2)
- U2 pad 6: Net-(U2-Pad6) -> Net-(J3-Pad4)
- U2 pad 7: Net-(U2-Pad7) -> Net-(J3-Pad5)
- U2 pad 9: Net-(N5-Pad0) -> Net-(N5-Pad9)
- U3 pad 1: Net-(N6-Pad4) -> Net-(N6-Pad5)
- U3 pad 10: (no net) -> Net-(N6-Pad0)
- U3 pad 16: Net-(N6-Pad5) -> Net-(N6-Pad4)
- U3 pad 3: Net-(U3-Pad3) -> Net-(J4-Pad1)
- U3 pad 4: GND -> Net-(J4-Pad2)
- U3 pad 6: Net-(U3-Pad6) -> Net-(J4-Pad4)
- U3 pad 7: Net-(U3-Pad7) -> Net-(J4-Pad5)
- U3 pad 8: (no net) -> Net-(N6-Pad8)
- U3 pad 9: Net-(N6-Pad0) -> Net-(N6-Pad9)
- U4 pad 1: Net-(N3-Pad4) -> Net-(N3-Pad5)
- U4 pad 10: Net-(N3-Pad9) -> Net-(N3-Pad0)
- U4 pad 16: Net-(N3-Pad5) -> Net-(N3-Pad4)
- U4 pad 3: Net-(U4-Pad3) -> Net-(J10-Pad1)
- U4 pad 4: Net-(U4-Pad4) -> Net-(J10-Pad2)
- U4 pad 6: Net-(U4-Pad6) -> Net-(J10-Pad4)
- U4 pad 7: Net-(U4-Pad7) -> Net-(J10-Pad5)
- U4 pad 9: Net-(N3-Pad0) -> Net-(N3-Pad9)
- U5 pad 1: Net-(U4-Pad6) -> Net-(J32-Pad1)
- U5 pad 11: Net-(J2-Pad7) -> /clock
- U5 pad 12: Net-(J2-Pad5) -> /latch
- U5 pad 14: Net-(U5-Pad14) -> Net-(U13-Pad9)
- U5 pad 15: Net-(U4-Pad7) -> (no net)
- U5 pad 2: Net-(U4-Pad4) -> Net-(J32-Pad2)
- U5 pad 3: Net-(U4-Pad3) -> Net-(J29-Pad5)
- U5 pad 4: Net-(U5-Pad4) -> Net-(J29-Pad4)
- U5 pad 5: Net-(U5-Pad5) -> Net-(J29-Pad2)
- U5 pad 6: Net-(Q2-Pad2) -> Net-(J29-Pad1)
- U5 pad 7: Net-(U5-Pad7) -> (no net)
- U5 pad 9: Net-(U1-Pad14) -> Net-(U11-Pad14)
- U6 pad 1: Net-(N4-Pad4) -> Net-(N4-Pad5)
- U6 pad 10: (no net) -> Net-(N4-Pad0)
- U6 pad 16: Net-(N4-Pad5) -> Net-(N4-Pad4)
- U6 pad 3: Net-(U5-Pad7) -> Net-(J11-Pad1)
- U6 pad 4: GND -> Net-(J11-Pad2)
- U6 pad 6: Net-(U5-Pad5) -> Net-(J11-Pad4)
- U6 pad 7: Net-(U5-Pad4) -> Net-(J11-Pad5)
- U6 pad 8: (no net) -> Net-(N4-Pad8)
- U6 pad 9: Net-(N4-Pad0) -> Net-(N4-Pad9)
- U7 pad 1: Net-(N1-Pad4) -> Net-(N1-Pad5)
- U7 pad 10: Net-(N1-Pad9) -> Net-(N1-Pad0)
- U7 pad 16: Net-(N1-Pad5) -> Net-(N1-Pad4)
- U7 pad 3: Net-(U1-Pad3) -> Net-(J12-Pad1)
- U7 pad 4: Net-(U1-Pad2) -> Net-(J12-Pad2)
- U7 pad 6: Net-(U1-Pad1) -> Net-(J12-Pad4)
- U7 pad 7: Net-(U1-Pad15) -> Net-(J12-Pad5)
- U7 pad 9: Net-(N1-Pad0) -> Net-(N1-Pad9)
- U8 pad 1: Net-(U2-Pad6) -> (no net)
- U8 pad 11: Net-(J2-Pad7) -> /clock
- U8 pad 12: Net-(J2-Pad5) -> /latch
- U8 pad 15: Net-(U2-Pad7) -> (no net)
- U8 pad 2: Net-(U2-Pad4) -> (no net)
- U8 pad 3: Net-(U2-Pad3) -> Net-(J27-Pad5)
- U8 pad 4: Net-(U3-Pad7) -> Net-(J27-Pad4)
- U8 pad 5: Net-(U3-Pad6) -> Net-(J27-Pad2)
- U8 pad 6: Net-(Q1-Pad2) -> Net-(J27-Pad1)
- U8 pad 7: Net-(U3-Pad3) -> (no net)
- U8 pad 9: Net-(U5-Pad14) -> Net-(U13-Pad14)
- U9 pad 1: (no net) -> Net-(N2-Pad5)
- U9 pad 10: (no net) -> Net-(N2-Pad0)
- U9 pad 11: (no net) -> Net-(N2-Pad7)
- U9 pad 13: (no net) -> Net-(N2-Pad6)
- U9 pad 16: (no net) -> Net-(N2-Pad4)
- U9 pad 3: Net-(U1-Pad7) -> Net-(J13-Pad2)
- U9 pad 4: GND -> Net-(J13-Pad3)
- U9 pad 6: Net-(U1-Pad5) -> Net-(J13-Pad5)
- U9 pad 7: GND -> Net-(J13-Pad6)
- U9 pad 8: (no net) -> Net-(N2-Pad8)
- U9 pad 9: Net-(N2-Pad0) -> Net-(N2-Pad9)
Routing:
- net Net-(J1-Pad1): track 246.7 -> 0.00 mm
- net Net-(J13-Pad1): track 0.00 -> 225.6 mm
- net Net-(J4-Pad1): track 210.1 -> 5.08 mm
- net VCC: track 249.3 -> 452.8 mm
- net /clock: track 0.00 -> 142.5 mm
- net /latch: track 0.00 -> 142.2 mm
- net Net-(J1-Pad2): track 0.00 -> 135.4 mm
- net Net-(J2-Pad7): track 123.3 -> 0.00 mm
- net Net-(J2-Pad5): track 121.8 -> 0.00 mm
- net Net-(U5-Pad14): track 39.7 -> 0.00 mm
- net Net-(Q4-Pad2): track 36.6 -> 0.00 mm
- net Net-(N2-Pad5): track 0.00 -> 36.0 mm
- net Net-(N4-Pad8): track 0.00 -> 27.5 mm
- net Net-(N6-Pad8): track 0.00 -> 27.4 mm
- net Net-(Q2-Pad2): track 26.2 -> 0.00 mm
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Other:
- board size 152.4 x 53.3 mm -> 167.6 x 104.1 mm
- net class Default: trace_width 0.5 -> 1
- rule trace_min: 0.5 -> 1

Commit message: Perfected design
Parts:
- removed J22, J6: CONN_01X01, Connectors:1pin
- added C1: C, Capacitors_THT:C_Disc_D4.3mm_W1.9mm_P5.00mm, F.Cu at (140.3, 87.0)
- added C2: CP, Capacitors_THT:CP_Radial_D8.0mm_P3.50mm, F.Cu at (116.8, 118.1)
- added C3: C, Capacitors_THT:C_Disc_D4.3mm_W1.9mm_P5.00mm, F.Cu at (128.3, 117.5)
- added C4: CP, Capacitors_THT:CP_Radial_D8.0mm_P3.50mm, F.Cu at (147.3, 86.0)
- added R1: 2.2k, Resistors_THT:R_Axial_DIN0207_L6.3mm_D2.5mm_P7.62mm_Horizontal, F.Cu at (78.7, 117.5)
- added R2: 2.2k, Resistors_THT:R_Axial_DIN0207_L6.3mm_D2.5mm_P7.62mm_Horizontal, F.Cu at (59.7, 117.5)
- moved Q1 3.81 mm to (85.1, 62.2)
- moved Q2 3.81 mm to (82.5, 62.2)
- moved Q3 3.81 mm to (135.9, 62.2)
- moved Q4 3.81 mm to (133.3, 62.2)
- moved R10 3.81 mm to (133.3, 52.1)
- moved R7 3.81 mm to (85.1, 52.1)
- moved R8 3.81 mm to (82.5, 52.1)
- moved R9 3.81 mm to (135.9, 52.1)
Routing:
- net Net-(N1-Pad8): track 0.00 -> 27.4 mm
- net VCC: track 452.8 -> 474.7 mm
- net Net-(N8-PadK): track 6.56 -> 0.00 mm
- net /data: track 13.0 -> 18.5 mm
- net Net-(J26-Pad2): track 21.3 -> 16.6 mm
- net Net-(J14-Pad2): track 21.3 -> 16.6 mm
- net Net-(N7-PadK): track 20.2 -> 16.4 mm
- net Net-(N10-PadK): track 6.56 -> 2.75 mm
- net Net-(N9-PadK): track 20.2 -> 16.5 mm
- net /latch: track 142.2 -> 145.2 mm
- net Net-(Q2-Pad1): track 5.08 -> 2.54 mm
- net Net-(Q1-Pad1): track 5.08 -> 2.54 mm
- net Net-(J14-Pad1): track 5.61 -> 4.34 mm
- net Net-(J26-Pad1): track 5.61 -> 4.34 mm

Commit message: Final fixes
Parts:
- removed J26: CONN_01X02, Pin_Headers:Pin_Header_Angled_1x02_Pitch2.54mm
- removed J28, J30: CONN_01X06, Socket_Strips:Socket_Strip_Straight_1x06_Pitch2.54mm
- removed J32, J33: CONN_01X02, Socket_Strips:Socket_Strip_Straight_1x02_Pitch2.54mm
- removed J7, J8: CONN_01X01, Connectors:1pin
- added J6: CONN_01X07, Pin_Headers:Pin_Header_Angled_1x07_Pitch2.54mm, B.Cu at (111.8, 66.0)
- C1, C2, C3, C4, J10, J12, J13, J3, R1, R2: moved to B.Cu
- J11: value CONN_01X06 -> CONN_01X07; footprint Pin_Headers:Pin_Header_Angled_1x06_Pitch2.54mm -> Socket_Strips:Socket_Strip_Straight_1x07_Pitch2.54mm; moved to B.Cu
- J14: value CONN_01X02 -> CONN_01X07; footprint Pin_Headers:Pin_Header_Angled_1x02_Pitch2.54mm -> Socket_Strips:Socket_Strip_Straight_1x07_Pitch2.54mm; moved to B.Cu
- J4: value CONN_01X06 -> CONN_01X07; footprint Pin_Headers:Pin_Header_Angled_1x06_Pitch2.54mm -> Pin_Headers:Pin_Header_Angled_1x07_Pitch2.54mm; moved to B.Cu
- moved J14 30.0 mm to (61.0, 90.2)
- moved J11 27.3 mm to (111.8, 90.2)
- moved R10 24.4 mm to (137.2, 27.9)
- moved R7 24.4 mm to (81.3, 27.9)
- moved R8 24.4 mm to (86.4, 27.9)
- moved R9 24.4 mm to (132.1, 27.9)
- moved J31 15.2 mm to (162.6, 90.2), turned to 270 degrees
- moved J13 15.2 mm to (162.6, 66.0)
- moved J5 12.7 mm to (139.7, 90.2), turned to 270 degrees
- moved J27 12.7 mm to (38.1, 90.2), turned to 270 degrees
- moved J29 12.7 mm to (88.9, 90.2), turned to 270 degrees
- moved J12 12.7 mm to (139.7, 66.0)
- moved J3 12.7 mm to (38.1, 66.0)
- moved J4 12.7 mm to (61.0, 66.0)
- moved J10 12.7 mm to (88.9, 66.0)
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Connections:
- J10 pad 3: VCC -> Net-(J10-Pad3)
- J10 pad 4: Net-(J10-Pad4) -> VCC
- J10 pad 6: GND -> Net-(J10-Pad6)
- J11 pad 1: Net-(J11-Pad1) -> GND
- J11 pad 3: VCC -> Net-(J11-Pad3)
- J11 pad 4: Net-(J11-Pad4) -> VCC
- J11 pad 6: GND -> Net-(J11-Pad6)
- J12 pad 3: VCC -> Net-(J12-Pad3)
- J12 pad 4: Net-(J12-Pad4) -> VCC
- J12 pad 6: GND -> Net-(J12-Pad6)
- J13 pad 1: Net-(J13-Pad1) -> GND
- J13 pad 7: GND -> Net-(J13-Pad7)
- J14 pad 1: Net-(J14-Pad1) -> GND
- J2 pad 2: (no net) -> Net-(J2-Pad2)
- J27 pad 1: Net-(J27-Pad1) -> GND
- J27 pad 3: VCC -> Net-(J27-Pad3)
- J27 pad 4: Net-(J27-Pad4) -> VCC
- J27 pad 6: GND -> Net-(J27-Pad6)
- J29 pad 3: VCC -> Net-(J29-Pad3)
- J29 pad 4: Net-(J29-Pad4) -> VCC
- J29 pad 6: GND -> Net-(J29-Pad6)
- J3 pad 1: Net-(J3-Pad1) -> GND
- J3 pad 3: VCC -> Net-(J3-Pad3)
- J3 pad 4: Net-(J3-Pad4) -> VCC
- J3 pad 6: GND -> Net-(J3-Pad6)
- J31 pad 1: Net-(J31-Pad1) -> GND
- J31 pad 7: GND -> Net-(J31-Pad7)
- J4 pad 1: Net-(J4-Pad1) -> GND
- J4 pad 3: VCC -> Net-(J4-Pad3)
- J4 pad 4: Net-(J4-Pad4) -> VCC
- J4 pad 6: GND -> Net-(J4-Pad6)
- J5 pad 3: VCC -> Net-(J5-Pad3)
- J5 pad 4: Net-(J5-Pad4) -> VCC
- J5 pad 6: GND -> Net-(J5-Pad6)
- J9 pad 3: (no net) -> Net-(J9-Pad3)
- J9 pad 5: Net-(J31-Pad1) -> Net-(J31-Pad7)
- N10 pad A: Net-(J13-Pad1) -> Net-(N10-PadA)
- N7 pad A: Net-(J13-Pad1) -> Net-(N7-PadA)
- N8 pad A: Net-(J13-Pad1) -> Net-(N8-PadA)
- N9 pad A: Net-(J13-Pad1) -> Net-(N9-PadA)
- Q1 pad 1: Net-(Q1-Pad1) -> Net-(N8-PadK)
- Q1 pad 2: Net-(J14-Pad2) -> Net-(J4-Pad7)
- Q2 pad 1: Net-(Q2-Pad1) -> Net-(N9-PadK)
- Q2 pad 2: Net-(J14-Pad1) -> Net-(J10-Pad1)
- Q3 pad 1: Net-(Q3-Pad1) -> Net-(N10-PadK)
- Q4 pad 1: Net-(Q4-Pad1) -> Net-(N7-PadK)
- Q4 pad 2: Net-(J26-Pad1) -> Net-(J12-Pad1)
- R10 pad 1: Net-(N7-PadK) -> Net-(J13-Pad7)
- R10 pad 2: Net-(Q4-Pad1) -> Net-(N7-PadA)
- R11 pad 1: Net-(J13-Pad1) -> Net-(J13-Pad7)
- R12 pad 1: Net-(J13-Pad1) -> Net-(J13-Pad7)
- R13 pad 1: Net-(J13-Pad1) -> Net-(J13-Pad7)
- R14 pad 1: Net-(J13-Pad1) -> Net-(J13-Pad7)
- R15 pad 1: Net-(J13-Pad1) -> Net-(J13-Pad7)
- R16 pad 1: Net-(J13-Pad1) -> Net-(J13-Pad7)
- R7 pad 1: Net-(N8-PadK) -> Net-(J13-Pad7)
- R7 pad 2: Net-(Q1-Pad1) -> Net-(N8-PadA)
- R8 pad 1: Net-(N9-PadK) -> Net-(J13-Pad7)
- R8 pad 2: Net-(Q2-Pad1) -> Net-(N9-PadA)
- R9 pad 1: Net-(N10-PadK) -> Net-(J13-Pad7)
- R9 pad 2: Net-(Q3-Pad1) -> Net-(N10-PadA)
- U1 pad 1: Net-(J33-Pad1) -> Net-(J11-Pad7)
- U1 pad 15: (no net) -> Net-(U1-Pad15)
- U1 pad 2: Net-(J33-Pad2) -> Net-(J5-Pad1)
- U1 pad 3: Net-(J5-Pad5) -> Net-(J5-Pad2)
- U1 pad 4: Net-(J5-Pad4) -> Net-(J5-Pad3)
- U1 pad 5: Net-(J5-Pad2) -> Net-(J5-Pad5)
- U1 pad 6: Net-(J5-Pad1) -> Net-(J5-Pad6)
- U1 pad 7: (no net) -> Net-(U1-Pad7)
- U11 pad 1: (no net) -> Net-(U11-Pad1)
- U11 pad 15: (no net) -> Net-(U11-Pad15)
- U11 pad 2: (no net) -> Net-(U11-Pad2)
- U11 pad 3: Net-(J30-Pad5) -> Net-(J11-Pad2)
- U11 pad 4: Net-(J30-Pad4) -> Net-(J11-Pad3)
- U11 pad 5: Net-(J30-Pad2) -> Net-(J11-Pad5)
- U11 pad 6: Net-(J30-Pad1) -> Net-(J11-Pad6)
- U11 pad 7: (no net) -> Net-(U11-Pad7)
- U13 pad 1: (no net) -> Net-(U13-Pad1)
- U13 pad 15: (no net) -> Net-(U13-Pad15)
- U13 pad 2: (no net) -> Net-(U13-Pad2)
- U13 pad 3: Net-(J28-Pad5) -> Net-(J14-Pad2)
- U13 pad 4: Net-(J28-Pad4) -> Net-(J14-Pad3)
- U13 pad 5: Net-(J28-Pad2) -> Net-(J14-Pad5)
- U13 pad 6: Net-(J28-Pad1) -> Net-(J14-Pad6)
- U13 pad 7: (no net) -> Net-(U13-Pad7)
- U14 pad 1: (no net) -> Net-(U14-Pad1)
- U14 pad 15: (no net) -> Net-(U14-Pad15)
- U14 pad 2: (no net) -> Net-(U14-Pad2)
- U14 pad 3: Net-(J31-Pad6) -> Net-(J31-Pad2)
- U14 pad 4: Net-(J31-Pad5) -> Net-(J31-Pad3)
- U14 pad 5: Net-(J31-Pad3) -> Net-(J31-Pad5)
- U14 pad 6: Net-(J31-Pad2) -> Net-(J31-Pad6)
- U14 pad 7: (no net) -> Net-(U14-Pad7)
- U14 pad 9: (no net) -> Net-(U14-Pad9)
- U2 pad 3: Net-(J3-Pad1) -> Net-(J3-Pad6)
- U2 pad 4: Net-(J3-Pad2) -> Net-(J3-Pad5)
- U2 pad 6: Net-(J3-Pad4) -> Net-(J3-Pad3)
- U2 pad 7: Net-(J3-Pad5) -> Net-(J3-Pad2)
- U3 pad 3: Net-(J4-Pad1) -> Net-(J4-Pad6)
- U3 pad 4: Net-(J4-Pad2) -> Net-(J4-Pad5)
- U3 pad 6: Net-(J4-Pad4) -> Net-(J4-Pad3)
- U3 pad 7: Net-(J4-Pad5) -> Net-(J4-Pad2)
- U4 pad 3: Net-(J10-Pad1) -> Net-(J10-Pad6)
- U4 pad 4: Net-(J10-Pad2) -> Net-(J10-Pad5)
- U4 pad 6: Net-(J10-Pad4) -> Net-(J10-Pad3)
- U4 pad 7: Net-(J10-Pad5) -> Net-(J10-Pad2)
- U5 pad 1: Net-(J32-Pad1) -> Net-(J14-Pad7)
- U5 pad 15: (no net) -> Net-(U5-Pad15)
- U5 pad 2: Net-(J32-Pad2) -> Net-(J29-Pad1)
- U5 pad 3: Net-(J29-Pad5) -> Net-(J29-Pad2)
- U5 pad 4: Net-(J29-Pad4) -> Net-(J29-Pad3)
- U5 pad 5: Net-(J29-Pad2) -> Net-(J29-Pad5)
- U5 pad 6: Net-(J29-Pad1) -> Net-(J29-Pad6)
- U5 pad 7: (no net) -> Net-(U5-Pad7)
- U6 pad 3: Net-(J11-Pad1) -> Net-(J6-Pad6)
- U6 pad 4: Net-(J11-Pad2) -> Net-(J6-Pad5)
- U6 pad 6: Net-(J11-Pad4) -> Net-(J6-Pad3)
- U6 pad 7: Net-(J11-Pad5) -> Net-(J6-Pad2)
- U7 pad 3: Net-(J12-Pad1) -> Net-(J12-Pad6)
- U7 pad 4: Net-(J12-Pad2) -> Net-(J12-Pad5)
- U7 pad 6: Net-(J12-Pad4) -> Net-(J12-Pad3)
- U7 pad 7: Net-(J12-Pad5) -> Net-(J12-Pad2)
- U8 pad 1: (no net) -> Net-(U8-Pad1)
- U8 pad 15: (no net) -> Net-(U8-Pad15)
- U8 pad 2: (no net) -> Net-(U8-Pad2)
- U8 pad 3: Net-(J27-Pad5) -> Net-(J27-Pad2)
- U8 pad 4: Net-(J27-Pad4) -> Net-(J27-Pad3)
- U8 pad 5: Net-(J27-Pad2) -> Net-(J27-Pad5)
- U8 pad 6: Net-(J27-Pad1) -> Net-(J27-Pad6)
- U8 pad 7: (no net) -> Net-(U8-Pad7)
- U9 pad 3: Net-(J13-Pad2) -> Net-(J13-Pad6)
- U9 pad 4: Net-(J13-Pad3) -> Net-(J13-Pad5)
- U9 pad 6: Net-(J13-Pad5) -> Net-(J13-Pad3)
- U9 pad 7: Net-(J13-Pad6) -> Net-(J13-Pad2)
Routing:
- net Net-(J13-Pad1): track 225.6 -> 0.00 mm
- net Net-(J13-Pad7): track 0.00 -> 198.0 mm
- net Net-(N2-Pad8): track 0.00 -> 27.5 mm
- net Net-(J14-Pad7): track 0.00 -> 24.0 mm
- net Net-(J32-Pad1): track 22.7 -> 0.00 mm
- net Net-(J32-Pad2): track 21.7 -> 0.00 mm
- net Net-(J28-Pad4): track 21.6 -> 0.00 mm
- net Net-(J28-Pad5): track 21.6 -> 0.00 mm
- net Net-(J28-Pad2): track 19.3 -> 0.00 mm
- net Net-(J27-Pad3): track 0.00 -> 19.0 mm
- net Net-(J28-Pad1): track 18.7 -> 0.00 mm
- net Net-(J27-Pad4): track 18.7 -> 0.00 mm
- net Net-(J14-Pad3): track 0.00 -> 18.4 mm
- net Net-(J27-Pad6): track 0.00 -> 17.9 mm
- net Net-(J27-Pad1): track 17.7 -> 0.00 mm
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Other:
- net class Default: clearance 0.2 -> 0.4
- rule trace_clearance: 0.2 -> 0.4
